File: hw-covers.kicad_pcb (KiCad board)
At the start: 2 copper layers, 122 x 70 mm, 117 parts, among them J1 Screw_Terminal_01x04, J10 Screw_Terminal_01x03, J11 Screw_Terminal_01x03, J2 Screw_Terminal_01x04, J3 Conn_01x04_Pin, J4 Conn_01x04_Pin, J5 Screw_Terminal_01x03, J6 Conn_01x02_Pin, J7 Screw_Terminal_01x04, J8 Screw_Terminal_01x03, J9 Screw_Terminal_01x03, K1 JRC-21F(4100), K10 JRC-21F(4100), K2 JRC-21F(4100), K3 JRC-21F(4100), K4 JRC-21F(4100), K5 JRC-21F(4100), K6 JRC-21F(4100), K7 JRC-21F(4100), K8 JRC-21F(4100), K9 JRC-21F(4100), Q1 PMBT3904235, Q10 PMBT3904235, Q11 PMBT3904235, Q2 PMBT3904235, Q3 PMBT3904235, Q4 PMBT3904235, Q5 PMBT3904235, Q6 PMBT3904235, Q7 PMBT3904235, Q8 PMBT3904235, Q9 PMBT3904235, SW1 SW_Push, U1 ESP32-S3-WROOM-1, U2 NCP1117-3.3_SOT223, U3 HLK-2M05

Commit message: Release 1.1
Parts:
- removed R16: 1k, Resistor_SMD:R_0402_1005Metric
- removed U3: HLK-2M05, guille-lib:HLK-2M05
- added PS1: HLK-2M05, Converter_ACDC:Converter_ACDC_Hi-Link_HLK-2Mxx, F.Cu at (108.8, 110.1)
- added R5: 1k, Resistor_SMD:R_0603_1608Metric, F.Cu at (132.9, 94.0)
- C1, C2: footprint Capacitor_SMD:C_1206_3216Metric -> Capacitor_SMD:C_0805_2012Metric
- C10, C11, C12, C13, C14, C4, C5, C6, C7, C8, C9: footprint Capacitor_SMD:C_0402_1005Metric -> Capacitor_SMD:C_0603_1608Metric
- D1, D10, D11, D12, D13, D2, D6, D7, D8, D9: footprint Diode_SMD:D_SOD-323 -> Diode_SMD:D_SOD-123
- K1, K10, K2, K3, K4, K5, K6, K7, K8, K9: value JRC-21F(4100) -> HF46F; footprint guille-lib:JRC-21F(4100) -> guille-lib:HF46F
- R1, R10, R11, R12, R13, R14, R15, R17, R18, R19, R2, R20, R21, R22, R23, R24, R25, R26, R27, R28, R29, R3, R30, R31, R32, R33, R34, R35, R36, R37, R4, R9: footprint Resistor_SMD:R_0402_1005Metric -> Resistor_SMD:R_0603_1608Metric
- moved Q1 95.5 mm to (119.7, 94.4)
- moved R2 95.3 mm to (117.2, 94.0)
- moved D2 92.7 mm to (118.8, 91.3)
- moved K1 90.9 mm to (121.2, 88.7), turned to 90 degrees
- moved K10 89.5 mm to (191.5, 88.7), turned to 90 degrees
- moved D13 86.4 mm to (189.2, 91.3)
- moved Q10 83.8 mm to (190.1, 94.4)
- moved R15 71.9 mm to (187.6, 94.0)
- moved K9 70.1 mm to (183.7, 88.7), turned to 90 degrees
- moved Q3 68.0 mm to (135.4, 94.4)
- moved D12 66.6 mm to (181.3, 91.3)
- moved D6 65.1 mm to (134.5, 91.3)
- moved Q9 64.1 mm to (182.2, 94.4)
- moved Q2 63.9 mm to (127.5, 94.4)
- moved K3 63.7 mm to (136.8, 88.7), turned to 90 degrees
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Connections:
- J1 pad 1: /OUT3_UP -> /OUT3_DOWN
- J1 pad 2: /OUT3_DOWN -> /OUT3_UP
- J1 pad 3: /OUT4_UP -> /OUT2_DOWN
- J1 pad 4: /OUT4_DOWN -> /OUT2_UP
- J2 pad 1: /OUT5_UP -> /OUT1_DOWN
- J2 pad 2: /OUT5_DOWN -> /OUT1_UP
- J7 pad 1: /OUT1_UP -> /OUT5_DOWN
- J7 pad 2: /OUT1_DOWN -> /OUT5_UP
- J7 pad 3: /OUT2_UP -> /OUT4_DOWN
- J7 pad 4: /OUT2_DOWN -> /OUT4_UP
- K1 pad 1: /LF -> /OUT1_UP
- K1 pad 2: +5V -> /LF
- K1 pad 3: unconnected-(K1-NC-Pad3) -> Net-(D2-A)
- K1 pad 4: /OUT1_UP -> +5V
- K10 pad 1: /LF -> /OUT5_DOWN
- K10 pad 2: +5V -> /LF
- K10 pad 3: unconnected-(K10-NC-Pad3) -> Net-(D13-A)
- K10 pad 4: /OUT5_DOWN -> +5V
- K2 pad 1: /LF -> /OUT1_DOWN
- K2 pad 2: +5V -> /LF
- K2 pad 3: unconnected-(K2-NC-Pad3) -> Net-(D1-A)
- K2 pad 4: /OUT2_UP -> +5V
- K3 pad 1: /LF -> /OUT2_UP
- K3 pad 2: +5V -> /LF
- K3 pad 3: unconnected-(K3-NC-Pad3) -> Net-(D6-A)
- K3 pad 4: /OUT1_DOWN -> +5V
- K4 pad 1: /LF -> /OUT2_DOWN
- K4 pad 2: +5V -> /LF
- K4 pad 3: unconnected-(K4-NC-Pad3) -> Net-(D7-A)
- K4 pad 4: /OUT2_DOWN -> +5V
- K5 pad 1: /LF -> /OUT3_UP
- K5 pad 2: +5V -> /LF
- K5 pad 3: unconnected-(K5-NC-Pad3) -> Net-(D8-A)
- K5 pad 4: /OUT3_UP -> +5V
- K6 pad 1: /LF -> /OUT3_DOWN
- K6 pad 2: +5V -> /LF
- K6 pad 3: unconnected-(K6-NC-Pad3) -> Net-(D9-A)
- K6 pad 4: /OUT4_UP -> +5V
- K7 pad 1: /LF -> /OUT4_UP
- K7 pad 2: +5V -> /LF
- K7 pad 3: unconnected-(K7-NC-Pad3) -> Net-(D10-A)
- K7 pad 4: /OUT3_DOWN -> +5V
- K8 pad 1: /LF -> /OUT4_DOWN
- K8 pad 2: +5V -> /LF
- K8 pad 3: unconnected-(K8-NC-Pad3) -> Net-(D11-A)
- K8 pad 4: /OUT4_DOWN -> +5V
- K9 pad 1: /LF -> /OUT5_UP
- K9 pad 2: +5V -> /LF
- K9 pad 3: unconnected-(K9-NC-Pad3) -> Net-(D12-A)
- K9 pad 4: /OUT5_UP -> +5V
- R1 pad 1: /2OUT1 -> /1OUT2
- R10 pad 1: /2OUT2 -> /3OUT1
- R10 pad 2: Net-(Q4-Pad1) -> Net-(Q5-Pad1)
- R11 pad 1: /3OUT1 -> /3OUT2
- R11 pad 2: Net-(Q5-Pad1) -> Net-(Q6-Pad1)
- R12 pad 2: Net-(Q6-Pad1) -> Net-(Q7-Pad1)
- R13 pad 1: /3OUT2 -> /4OUT2
- R13 pad 2: Net-(Q7-Pad1) -> Net-(Q8-Pad1)
- R14 pad 1: /4OUT2 -> /5OUT1
- R14 pad 2: Net-(Q8-Pad1) -> Net-(Q9-Pad1)
- R15 pad 1: /5OUT1 -> /5OUT2
- R15 pad 2: Net-(Q9-Pad1) -> Net-(Q10-Pad1)
- R9 pad 1: /1OUT2 -> /2OUT2
- R9 pad 2: Net-(Q3-Pad1) -> Net-(Q4-Pad1)
- U1 pad 10: /1OUT2 -> /4OUT1
- U1 pad 11: /2OUT1 -> /3OUT2
- U1 pad 12: /2OUT2 -> /3OUT1
- U1 pad 13: /3OUT1 -> /2OUT2
- U1 pad 14: /3OUT2 -> /2OUT1
- U1 pad 17: /4OUT1 -> /1OUT2
- U1 pad 18: /4OUT2 -> /1OUT1
- U1 pad 19: /5OUT1 -> /LED1
- U1 pad 20: /5OUT2 -> /LED2
- U1 pad 7: /LED2 -> /5OUT2
- U1 pad 8: /LED1 -> /5OUT1
- U1 pad 9: /1OUT1 -> /4OUT2
Routing:
- net /5OUT2: track 89.6 -> 9.09 mm
- net +3V3: track 142.4 -> 213.2 mm, vias 2 -> 12
- net /5OUT1: track 78.8 -> 12.4 mm
- net +5V: track 290.1 -> 224.6 mm, vias 1 -> 0
- net /4OUT2: track 68.1 -> 18.5 mm
- net /1OUT2: track 17.1 -> 59.7 mm
- net /1OUT1: track 26.0 -> 68.2 mm
- net /OUT5_DOWN: track 50.3 -> 11.5 mm
- net /OUT5_UP: track 41.7 -> 10.4 mm
- net /4OUT1: track 57.3 -> 26.5 mm
- net /IR: track 7.50 -> 38.3 mm
- net /OUT4_DOWN: track 38.6 -> 9.22 mm
- net /ESP_RX: track 39.4 -> 10.3 mm
- net /LF: track 165.4 -> 137.1 mm
- net /ESP_TX: track 38.9 -> 10.8 mm
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Other:
- board size 122 x 70 mm -> 100 x 90 mm
- board text added: "1DN 1UP N L"
- board text added: "2UP 2DN 3UP 3DN"
- board text added: "3DN 3UP 2DN 2UP"
- board text added: "4UP 4DN 5UP 5DN"
- board text added: "5DN 5UP 4DN 4UP"
- board text added: "GPIO0"
- board text added: "IR- IR+"
- board text added: "L N 1UP 1DN"
- board text added: "MAR 2025"
- board text added: "Rev 1.1"
- board text removed: "1UP 1DN 2UP 2DN"
- board text removed: "2DN 2UP 1DN 1UP"
- board text removed: "3 R T G"
- board text removed: "3UP 3DN 4UP 4DN"
- board text removed: "4DN 4UP 3DN 3UP"
- board text removed: "5UP 5DN N L"
- board text removed: "FEB 2025"
- board text removed: "L N 5DN 5UP"
- board text removed: "Rev 1.0"

Commit message: Minor changes to release 1.1
Routing:
- net GND: vias 160 -> 175
Changed lines of the file:
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@@
 	)
 	(via
+		(at 183 135)
+		(size 0.6)
+		(drill 0.3)
+		(layers "F.Cu" "B.Cu")
+		(free yes)
+		(net 1)
+	)
+	(via
 		(at 131 99)
 		(size 0.6)
@@
 	)
 	(via
+		(at 196 125)
+		(size 0.6)
+		(drill 0.3)
+		(layers "F.Cu" "B.Cu")
+		(free yes)
+		(net 1)
+	)
+	(via
 		(at 155 128)
 		(size 0.6)
@@
 	)
 	(via
+		(at 120 106)
+		(size 0.6)
+		(drill 0.3)
+		(layers "F.Cu" "B.Cu")
+		(free yes)
+		(net 1)
+	)
+	(via
 		(at 184 110)
 		(size 0.6)
@@
 	)
 	(via
+		(at 202 68)
+		(size 0.6)
+		(drill 0.3)
+		(layers "F.Cu" "B.Cu")
+		(free yes)
+		(net 1)
+	)
+	(via
 		(at 155 102)
 		(size 0.6)
@@
 	)
 	(via
+		(at 202 66)
+		(size 0.6)
+		(drill 0.3)
+		(layers "F.Cu" "B.Cu")
+		(free yes)
+		(net 1)
+	)
+	(via
 		(at 163 102)
 		(size 0.6)
@@
 	)
 	(via
+		(at 183 139)
+		(size 0.6)
+		(drill 0.3)
+		(layers "F.Cu" "B.Cu")
+		(free yes)
+		(net 1)
+	)
+	(via
 		(at 193 93)
 		(size 0.6)
@@
 	)
 	(via
+		(at 120 108)
+		(size 0.6)
+		(drill 0.3)
+		(layers "F.Cu" "B.Cu")
+		(free yes)
+		(net 1)
+	)
+	(via
 		(at 182 112)
 		(size 0.6)
@@
 	)
 	(via
+		(at 120 112)
+		(size 0.6)
+		(drill 0.3)
+		(layers "F.Cu" "B.Cu")
+		(free yes)
+		(net 1)
+	)
+	(via
 		(at 145 102)
 		(size 0.6)
@@
 	)
 	(via
+		(at 202 70)
+		(size 0.6)
+		(drill 0.3)
+		(layers "F.Cu" "B.Cu")
+		(free yes)
+		(net 1)
+	)
+	(via
 		(at 127 128)
 		(size 0.6)
@@
 	)
 	(via
+		(at 202 72)
+		(size 0.6)
+		(drill 0.3)
+		(layers "F.Cu" "B.Cu")
+		(free yes)
+		(net 1)
+	)
+	(via
 		(at 188 116)
 		(size 0.6)
@@
 	)
 	(via
+		(at 120 110)
+		(size 0.6)
+		(drill 0.3)
+		(layers "F.Cu" "B.Cu")
+		(free yes)
+		(net 1)
+	)
+	(via
 		(at 195 89)
 		(size 0.6)
@@
 	)
 	(via
+		(at 183 133)
+		(size 0.6)
+		(drill 0.3)
+		(layers "F.Cu" "B.Cu")
+		(free yes)
+		(net 1)
+	)
+	(via
 		(at 203 129)
 		(size 0.6)
@@
 	)
 	(via
+		(at 196 123)
+		(size 0.6)
+		(drill 0.3)
+		(layers "F.Cu" "B.Cu")
+		(free yes)
+		(net 1)
+	)
+	(via
 		(at 127 109.5)
 		(size 0.6)
@@
 	)
 	(via
+		(at 183 131)
+		(size 0.6)
+		(drill 0.3)
+		(layers "F.Cu" "B.Cu")
+		(free yes)
+		(net 1)
+	)
+	(via
 		(at 182 118)
 		(size 0.6)
@@
 	)
 	(via
+		(at 183 137)
+		(size 0.6)
+		(drill 0.3)
+		(layers "F.Cu" "B.Cu")
+		(free yes)
+		(net 1)
+	)
+	(via
 		(at 153 97)
 		(size 0.6)
@@
 		(polygon
 			(pts
-				(xy 119 103) (xy 115 99) (xy 115 86.5) (xy 190 86) (xy 194 82) (xy 194 61) (xy 204 61) (xy 204 141)
+				(xy 119 103) (xy 115 99) (xy 115 86) (xy 190 86) (xy 194 82) (xy 194 61) (xy 204 61) (xy 204 141)
 				(xy 104 141) (xy 104 127) (xy 119 112)
 			)

Commit message: Sch update for rev 2
Parts:
- removed D10, D11, D12, D13, D2, D6, D7, D8, D9: 1N4448W, Diode_SMD:D_SOD-123
- removed D5: LED, LED_SMD:LED_0603_1608Metric
- removed K1, K10, K2, K3, K4, K5, K6, K7, K8, K9: HF46F, guille-lib:HF46F
- removed Q1, Q10, Q2, Q3, Q4, Q5, Q6, Q7, Q8, Q9: PMBT3904235, Package_TO_SOT_SMD:SOT-23
- removed R1, R10, R11, R12, R13, R14, R15, R2, R5, R9: 1k, Resistor_SMD:R_0603_1608Metric
- removed RV1: Varistor, Varistor:RV_Disc_D12mm_W4.5mm_P7.5mm
- added C15: C, Capacitor_THT:C_Rect_L18.0mm_W7.0mm_P15.00mm_FKS3_FKP3, F.Cu at (106.8, 27.3)
- added C16: C, Capacitor_THT:C_Rect_L18.0mm_W7.0mm_P15.00mm_FKS3_FKP3, F.Cu at (106.8, 35.9)
- added C17: C, Capacitor_THT:C_Rect_L18.0mm_W7.0mm_P15.00mm_FKS3_FKP3, F.Cu at (106.8, 44.4)
- added C18: C, Capacitor_THT:C_Rect_L18.0mm_W7.0mm_P15.00mm_FKS3_FKP3, F.Cu at (106.8, 53.0)
- added C19: C, Capacitor_THT:C_Rect_L18.0mm_W7.0mm_P15.00mm_FKS3_FKP3, F.Cu at (106.8, 61.5)
- added C20: C, Capacitor_THT:C_Rect_L18.0mm_W7.0mm_P15.00mm_FKS3_FKP3, F.Cu at (106.8, 70.1)
- added C21: C, Capacitor_THT:C_Rect_L18.0mm_W7.0mm_P15.00mm_FKS3_FKP3, F.Cu at (106.8, 78.6)
- added C22: C, Capacitor_THT:C_Rect_L18.0mm_W7.0mm_P15.00mm_FKS3_FKP3, F.Cu at (106.8, 87.2)
- added C23: C, Capacitor_THT:C_Rect_L18.0mm_W7.0mm_P15.00mm_FKS3_FKP3, F.Cu at (106.8, 95.7)
- added C24: C, Capacitor_THT:C_Rect_L18.0mm_W7.0mm_P15.00mm_FKS3_FKP3, F.Cu at (106.8, 104.3)
- added D14: 1N4448W, Diode_SMD:D_SOD-123, F.Cu at (202.4, 24.7)
- added D24: 1N4448W, Diode_SMD:D_SOD-123, F.Cu at (202.4, 28.1)
- added D26: 1N4448W, Diode_SMD:D_SOD-123, F.Cu at (202.4, 31.4)
- added D27: 1N4448W, Diode_SMD:D_SOD-123, F.Cu at (202.4, 34.8)
- added D28: 1N4448W, Diode_SMD:D_SOD-123, F.Cu at (202.4, 38.1)
- added D29: 1N4448W, Diode_SMD:D_SOD-123, F.Cu at (202.4, 41.5)
- added D30: 1N4448W, Diode_SMD:D_SOD-123, F.Cu at (202.4, 44.8)
- added D31: 1N4448W, Diode_SMD:D_SOD-123, F.Cu at (202.4, 48.2)
- added D32: 1N4448W, Diode_SMD:D_SOD-123, F.Cu at (202.4, 51.5)
- added D33: 1N4448W, Diode_SMD:D_SOD-123, F.Cu at (202.4, 54.9)
- added K11: SANYOU_SRD_Form_C, Relay_THT:Relay_SPDT_SANYOU_SRD_Series_Form_C, F.Cu at (126.1, 31.5)
- added K12: SANYOU_SRD_Form_C, Relay_THT:Relay_SPDT_SANYOU_SRD_Series_Form_C, F.Cu at (126.1, 48.5)
- added K13: SANYOU_SRD_Form_C, Relay_THT:Relay_SPDT_SANYOU_SRD_Series_Form_C, F.Cu at (126.1, 65.4)
- added K14: SANYOU_SRD_Form_C, Relay_THT:Relay_SPDT_SANYOU_SRD_Series_Form_C, F.Cu at (126.1, 82.4)
- added K15: SANYOU_SRD_Form_C, Relay_THT:Relay_SPDT_SANYOU_SRD_Series_Form_C, F.Cu at (126.1, 99.3)
- added K16: SANYOU_SRD_Form_C, Relay_THT:Relay_SPDT_SANYOU_SRD_Series_Form_C, F.Cu at (147.3, 31.5)
- added K17: SANYOU_SRD_Form_C, Relay_THT:Relay_SPDT_SANYOU_SRD_Series_Form_C, F.Cu at (147.3, 48.5)
- added K18: SANYOU_SRD_Form_C, Relay_THT:Relay_SPDT_SANYOU_SRD_Series_Form_C, F.Cu at (147.3, 65.4)
- added K19: SANYOU_SRD_Form_C, Relay_THT:Relay_SPDT_SANYOU_SRD_Series_Form_C, F.Cu at (147.3, 82.4)
- added K20: SANYOU_SRD_Form_C, Relay_THT:Relay_SPDT_SANYOU_SRD_Series_Form_C, F.Cu at (147.3, 99.3)
- added Q12: PMBT3904235, Package_TO_SOT_SMD:SOT-23, F.Cu at (188.4, 79.8)
- added Q13: PMBT3904235, Package_TO_SOT_SMD:SOT-23, F.Cu at (188.4, 84.2)
- added Q14: PMBT3904235, Package_TO_SOT_SMD:SOT-23, F.Cu at (188.4, 88.7)
- added Q15: PMBT3904235, Package_TO_SOT_SMD:SOT-23, F.Cu at (188.4, 93.1)
- added Q16: PMBT3904235, Package_TO_SOT_SMD:SOT-23, F.Cu at (188.4, 97.6)
- added Q17: PMBT3904235, Package_TO_SOT_SMD:SOT-23, F.Cu at (193.3, 79.8)
- added Q18: PMBT3904235, Package_TO_SOT_SMD:SOT-23, F.Cu at (193.3, 84.2)
- added Q19: PMBT3904235, Package_TO_SOT_SMD:SOT-23, F.Cu at (193.3, 88.7)
- added Q20: PMBT3904235, Package_TO_SOT_SMD:SOT-23, F.Cu at (193.3, 93.1)
- added Q21: PMBT3904235, Package_TO_SOT_SMD:SOT-23, F.Cu at (193.3, 97.6)
- added R16: 1k, Resistor_SMD:R_0603_1608Metric, F.Cu at (197.8, 78.8)
- added R38: 1k, Resistor_SMD:R_0603_1608Metric, F.Cu at (197.8, 81.3)
- added R39: R, Resistor_THT:R_Axial_DIN0614_L14.3mm_D5.7mm_P15.24mm_Horizontal, F.Cu at (168.5, 26.7)
- added R40: R, Resistor_THT:R_Axial_DIN0614_L14.3mm_D5.7mm_P15.24mm_Horizontal, F.Cu at (168.5, 33.9)
- added R41: 1k, Resistor_SMD:R_0603_1608Metric, F.Cu at (197.8, 83.8)
- added R42: 1k, Resistor_SMD:R_0603_1608Metric, F.Cu at (197.8, 86.3)
- added R43: R, Resistor_THT:R_Axial_DIN0614_L14.3mm_D5.7mm_P15.24mm_Horizontal, F.Cu at (168.5, 41.2)
- added R44: R, Resistor_THT:R_Axial_DIN0614_L14.3mm_D5.7mm_P15.24mm_Horizontal, F.Cu at (168.5, 48.4)
- added R45: 1k, Resistor_SMD:R_0603_1608Metric, F.Cu at (197.8, 88.8)
- added R46: 1k, Resistor_SMD:R_0603_1608Metric, F.Cu at (201.8, 78.8)
- added R47: 1k, Resistor_SMD:R_0603_1608Metric, F.Cu at (201.8, 81.3)
- added R48: 1k, Resistor_SMD:R_0603_1608Metric, F.Cu at (201.8, 83.8)
- added R49: R, Resistor_THT:R_Axial_DIN0614_L14.3mm_D5.7mm_P15.24mm_Horizontal, F.Cu at (168.5, 55.7)
- added R50: R, Resistor_THT:R_Axial_DIN0614_L14.3mm_D5.7mm_P15.24mm_Horizontal, F.Cu at (168.5, 62.9)
- added R51: R, Resistor_THT:R_Axial_DIN0614_L14.3mm_D5.7mm_P15.24mm_Horizontal, F.Cu at (168.5, 70.2)
- added R52: R, Resistor_THT:R_Axial_DIN0614_L14.3mm_D5.7mm_P15.24mm_Horizontal, F.Cu at (168.5, 77.4)
- added R53: 1k, Resistor_SMD:R_0603_1608Metric, F.Cu at (201.8, 86.3)
- added R54: 1k, Resistor_SMD:R_0603_1608Metric, F.Cu at (201.8, 88.8)
- added R55: R, Resistor_THT:R_Axial_DIN0614_L14.3mm_D5.7mm_P15.24mm_Horizontal, F.Cu at (168.5, 84.7)
- added R56: R, Resistor_THT:R_Axial_DIN0614_L14.3mm_D5.7mm_P15.24mm_Horizontal, F.Cu at (168.5, 91.9)
- added RV10: Varistor, Varistor:RV_Disc_D12mm_W3.9mm_P7.5mm, F.Cu at (189.0, 68.7)
- added RV11: Varistor, Varistor:RV_Disc_D12mm_W3.9mm_P7.5mm, F.Cu at (189.0, 74.1)
- added RV12: Varistor, Varistor:RV_Disc_D12mm_W4.5mm_P7.5mm, F.Cu at (122.5, 176.2)
- added RV2: Varistor, Varistor:RV_Disc_D12mm_W3.9mm_P7.5mm, F.Cu at (189.0, 25.1)
- added RV3: Varistor, Varistor:RV_Disc_D12mm_W3.9mm_P7.5mm, F.Cu at (189.0, 30.5)
- added RV4: Varistor, Varistor:RV_Disc_D12mm_W3.9mm_P7.5mm, F.Cu at (189.0, 36.0)
- added RV5: Varistor, Varistor:RV_Disc_D12mm_W3.9mm_P7.5mm, F.Cu at (189.0, 41.4)
- added RV6: Varistor, Varistor:RV_Disc_D12mm_W3.9mm_P7.5mm, F.Cu at (189.0, 46.9)
- added RV7: Varistor, Varistor:RV_Disc_D12mm_W3.9mm_P7.5mm, F.Cu at (189.0, 52.3)
- added RV8: Varistor, Varistor:RV_Disc_D12mm_W3.9mm_P7.5mm, F.Cu at (189.0, 57.8)
- added RV9: Varistor, Varistor:RV_Disc_D12mm_W3.9mm_P7.5mm, F.Cu at (189.0, 63.2)
- D1: value 1N4448W -> LED; footprint Diode_SMD:D_SOD-123 -> LED_SMD:LED_0603_1608Metric
- R17: value 1k -> 180
- moved J6 142.3 mm to (106.8, 173.8), turned to 0 degrees
- moved Q11 137.5 mm to (111.5, 173.7), turned to 0 degrees
- moved H3 129.3 mm to (158.0, 173.9)
- moved F1 119.9 mm to (147.2, 176.5), turned to 0 degrees
- moved H1 111.6 mm to (158.0, 158.0)
- moved R17 106.8 mm to (164.0, 170.3), turned to 0 degrees
- moved J7 102.1 mm to (124.0, 143.0), turned to 0 degrees
- moved TP2 100.1 mm to (106.3, 183.9)
- moved TP1 91.7 mm to (106.3, 180.4)
- moved J3 85.0 mm to (146.1, 140.8)
- moved U2 72.1 mm to (137.9, 178.3), turned to 0 degrees
- moved J11 70.3 mm to (108.2, 162.4)
- moved R4 69.2 mm to (164.0, 160.3)
- moved J2 68.7 mm to (124.0, 128.5), turned to 0 degrees
- moved H4 67.4 mm to (158.0, 181.8)
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Connections:
- net /IN1_DOWN renamed /IN1_DN
- net /IN2_DOWN renamed /IN2_DN
- net /IN3_DOWN renamed /IN3_DN
- net /IN4_DOWN renamed /IN4_DN
- net /IN5_DOWN renamed /IN5_DN
- D1 pad 1: +5V -> Net-(D1-K)
- D1 pad 2: Net-(D1-A) -> +3V3
- D3 pad 2: +3V3 -> /LED1
- D4 pad 2: /LED1 -> /LED2
- J1 pad 1: /OUT3_DOWN -> /OUT3_DN
- J1 pad 3: /OUT2_DOWN -> /OUT2_DN
- J2 pad 1: /OUT1_DOWN -> /OUT1_DN
- J7 pad 1: /OUT5_DOWN -> /OUT5_DN
- J7 pad 3: /OUT4_DOWN -> /OUT4_DN
- R18 pad 2: /1IN1 -> /1IN2
- R19 pad 1: /1IN1 -> /1IN2
- R20 pad 1: /1IN2 -> /1IN1
- R21 pad 2: /1IN2 -> /1IN1
- R22 pad 1: /2IN1 -> /2IN2
- R23 pad 2: /2IN1 -> /2IN2
- R24 pad 1: /2IN2 -> /2IN1
- R25 pad 2: /2IN2 -> /2IN1
- R26 pad 1: /3IN1 -> /3IN2
- R27 pad 2: /3IN1 -> /3IN2
- R28 pad 1: /3IN2 -> /3IN1
- R29 pad 2: /3IN2 -> /3IN1
- R30 pad 1: /4IN1 -> /4IN2
- R31 pad 2: /4IN1 -> /4IN2
- R32 pad 1: /4IN2 -> /4IN1
- R33 pad 2: /4IN2 -> /4IN1
- R34 pad 1: /5IN1 -> /5IN2
- R35 pad 2: /5IN1 -> /5IN2
- R36 pad 1: /5IN2 -> /5IN1
- R37 pad 2: /5IN2 -> /5IN1
- R6 pad 1: Net-(D3-K) -> Net-(D1-K)
- R7 pad 1: Net-(D4-K) -> Net-(D3-K)
- R8 pad 1: Net-(D5-K) -> Net-(D4-K)
- U1 pad 10: /4OUT1 -> /DIR4
- U1 pad 11: /3OUT2 -> /OUT3
- U1 pad 12: /3OUT1 -> /DIR3
- U1 pad 13: /2OUT2 -> /OUT2
- U1 pad 14: /2OUT1 -> /DIR2
- U1 pad 17: /1OUT2 -> /OUT1
- U1 pad 18: /1OUT1 -> /DIR1
- U1 pad 7: /5OUT2 -> /OUT5
- U1 pad 8: /5OUT1 -> /DIR5
- U1 pad 9: /4OUT2 -> /OUT4
Routing:
- net +5V: track 224.6 -> 0.00 mm
- net +3V3: track 213.2 -> 0.00 mm, vias 12 -> 0
- net /LF: track 137.1 -> 0.00 mm
- net /1OUT1: track 68.2 -> 0.00 mm
- net /1IN1: track 66.9 -> 0.00 mm
- net /N: track 62.3 -> 0.00 mm
- net /1IN2: track 62.2 -> 0.00 mm
- net /1OUT2: track 59.7 -> 0.00 mm
- net /2IN1: track 51.7 -> 0.00 mm
- net /2OUT1: track 51.1 -> 0.00 mm
- net /2IN2: track 47.2 -> 0.00 mm
- net /3IN1: track 46.5 -> 0.00 mm
- net /2OUT2: track 44.7 -> 0.00 mm
- net /3IN2: track 43.6 -> 0.00 mm
- net /IR: track 38.3 -> 0.00 mm
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- removed copper zone on B.Cu, net GND
- removed copper zone on F.Cu, net GND
Other:
- board outline removed

Commit message: Add placement
Parts:
- R19, R20, R22, R24, R26, R28, R30, R32, R34, R36: value 10k -> 1k5
- moved D32 152.0 mm to (62.5, 111.0)
- moved H1 148.9 mm to (56.0, 49.5)
- moved R53 141.1 mm to (63.3, 113.1)
- moved D24 136.4 mm to (94.0, 111.0)
- moved D33 136.0 mm to (78.5, 111.0)
- moved F1 132.1 mm to (119.0, 47.5), turned to 180 degrees
- moved H2 128.6 mm to (211.5, 49.0)
- moved Q20 127.8 mm to (67.0, 112.1), turned to 90 degrees
- moved RV10 126.7 mm to (62.2, 66.8)
- moved D14 126.2 mm to (110.3, 111.0)
- moved R54 124.6 mm to (79.5, 113.0)
- moved RV12 122.6 mm to (102.6, 55.2), turned to 90 degrees
- moved J7 115.0 mm to (198.7, 55.5), turned to 180 degrees
- moved PS1 112.6 mm to (95.0, 55.2), turned to 180 degrees
- moved RV11 111.3 mm to (77.9, 66.8)
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
Commit message: Change in R values and routing test
Parts:
- moved J4 39.7 mm to (201.0, 131.5)
- moved J6 14.9 mm to (215.5, 129.1)
- moved Q11 14.8 mm to (210.8, 131.5)
- moved R17 13.9 mm to (210.3, 128.2)
- moved J1 11.7 mm to (163.4, 55.2)
- moved J7 11.7 mm to (187.0, 55.2)
- moved J2 11.2 mm to (139.8, 55.2)
- moved F1 10.6 mm to (112.0, 55.5)
- moved C1 7.45 mm to (59.9, 123.5), turned to -90 degrees
- moved C2 5.99 mm to (69.4, 123.4), turned to 90 degrees
- moved U2 4.13 mm to (64.7, 126.2), turned to -90 degrees
- moved R45 1.51 mm to (159.5, 114.1)
- moved R42 1.42 mm to (143.5, 114.1)
- moved R41 1.40 mm to (127.5, 114.1)
- moved R48 1.23 mm to (207.5, 114.1)
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Connections:
- J1 pad 1: /OUT3_DN -> /OUT3_UP
- J1 pad 2: /OUT3_UP -> /OUT3_DN
- J1 pad 3: /OUT2_DN -> /OUT2_UP
- J1 pad 4: /OUT2_UP -> /OUT2_DN
- J2 pad 1: /OUT1_DN -> /OUT1_UP
- J2 pad 2: /OUT1_UP -> /OUT1_DN
- J7 pad 1: /OUT5_DN -> /OUT5_UP
- J7 pad 2: /OUT5_UP -> /OUT5_DN
- J7 pad 3: /OUT4_DN -> /OUT4_UP
- J7 pad 4: /OUT4_UP -> /OUT4_DN
Routing:
- net +5V: track 0.00 -> 366.4 mm
- net /N: track 0.00 -> 273.8 mm
- net /LF: track 0.00 -> 175.1 mm
- net +3V3: track 0.00 -> 109.1 mm
- net /DIR1: track 0.00 -> 108.1 mm
- net /OUT1_DN: track 0.00 -> 105.3 mm
- net /OUT1_UP: track 0.00 -> 96.4 mm
- net /OUT1: track 0.00 -> 91.5 mm
- net GND: track 0.00 -> 90.0 mm
- net /OUT2_DN: track 0.00 -> 87.2 mm
- net /OUT2_UP: track 0.00 -> 78.2 mm
- net /DIR2: track 0.00 -> 75.8 mm
- net /OUT3_DN: track 0.00 -> 67.1 mm
- net /1IN2: track 0.00 -> 64.9 mm
- net /OUT3_UP: track 0.00 -> 56.8 mm
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
Commit message: Finish routing
Parts:
- TP1, TP2: moved to B.Cu
- moved TP2 20.6 mm to (174.8, 126.5), turned to 180 degrees
- moved TP1 19.3 mm to (177.5, 126.5), turned to 180 degrees
- moved J3 14.2 mm to (203.2, 132.7)
- moved R8 5.98 mm to (214.3, 124.6)
- moved R7 5.93 mm to (214.3, 122.5)
- moved R6 5.91 mm to (214.3, 120.4)
- moved D4 5.61 mm to (210.4, 124.7), turned to 180 degrees
- moved D3 5.55 mm to (210.4, 122.5), turned to 180 degrees
- moved D1 5.53 mm to (210.4, 120.4), turned to 180 degrees
- moved H4 3.81 mm to (215.0, 140.0)
- moved C1 3.70 mm to (63.6, 123.3)
- moved U2 3.70 mm to (68.4, 126.0)
- moved C2 3.70 mm to (73.1, 123.3)
- moved H2 3.64 mm to (215.0, 48.0)
- moved J4 3.23 mm to (198.0, 132.7)
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Connections:
- TP1 pad 1: Net-(U1-IO13) -> Net-(U1-IO48)
- U1 pad 10: /DIR4 -> /DIR5
- U1 pad 11: /OUT3 -> /OUT4
- U1 pad 12: /DIR3 -> /DIR4
- U1 pad 13: /OUT2 -> /2IN1
- U1 pad 14: /DIR2 -> /2IN2
- U1 pad 17: /OUT1 -> /1IN1
- U1 pad 18: /DIR1 -> /1IN2
- U1 pad 19: /LED1 -> /DIR1
- U1 pad 20: /LED2 -> /OUT1
- U1 pad 21: Net-(U1-IO13) -> /DIR2
- U1 pad 22: /1IN1 -> /OUT2
- U1 pad 23: /1IN2 -> /DIR3
- U1 pad 24: /2IN1 -> /OUT3
- U1 pad 25: /2IN2 -> Net-(U1-IO48)
- U1 pad 32: /3IN1 -> /3IN2
- U1 pad 33: /3IN2 -> /3IN1
- U1 pad 34: /4IN1 -> /4IN2
- U1 pad 35: /4IN2 -> /4IN1
- U1 pad 38: /5IN1 -> /5IN2
- U1 pad 39: /5IN2 -> /5IN1
- U1 pad 4: /EXT2 -> /EXT1
- U1 pad 5: /EXT1 -> /EXT2
- U1 pad 7: /OUT5 -> /LED2
- U1 pad 8: /DIR5 -> /LED1
- U1 pad 9: /OUT4 -> /OUT5
Routing:
- net +3V3: track 109.1 -> 272.1 mm, vias 0 -> 13
- net /LF: track 175.1 -> 288.1 mm
- net /2IN1: track 35.1 -> 89.8 mm, vias 0 -> 2
- net /2IN2: track 41.7 -> 94.6 mm, vias 0 -> 2
- net /1IN1: track 52.8 -> 101.4 mm, vias 0 -> 2
- net +5V: track 366.4 -> 408.3 mm, vias 0 -> 1
- net /1IN2: track 64.9 -> 104.4 mm, vias 0 -> 2
- net /DIR4: track 0.00 -> 39.3 mm
- net /N: track 273.8 -> 304.5 mm
- net /ESP_IO0: track 0.00 -> 29.8 mm, vias 0 -> 2
- net /ESP_TX: track 0.00 -> 29.0 mm, vias 0 -> 1
- net /ESP_RX: track 0.00 -> 28.5 mm, vias 0 -> 1
- net /5IN1: track 1.83 -> 29.3 mm
- net /EXT2: track 0.00 -> 26.6 mm
- net /OUT4: track 0.00 -> 25.7 mm
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- added copper zone on B.Cu, net GND
- added copper zone on F.Cu, net GND
Other:
- board outline added: 167 x 100 mm

Commit message: Finish PCB
Routing:
- net GND: track 97.1 -> 101.6 mm, vias 0 -> 223
- net +3V3: track 272.1 -> 274.0 mm
- net +5V: track 408.3 -> 407.0 mm
Other:
- board text added: "1UP 1DN N L"
- board text added: "2DN 2UP 3DN 3UP"
- board text added: "3UP 3DN 2UP 2DN"
- board text added: "4DN 4UP 5DN 5UP"
- board text added: "5UP 5DN 4UP 4DN"
- board text added: "MAR 2026"
- board text added: "N L 1DN 1UP"
- board text added: "Rev 2.0"
- board text removed: "1DN 1UP N L"
- board text removed: "2UP 2DN 3UP 3DN"
- board text removed: "3DN 3UP 2DN 2UP"
- board text removed: "4UP 4DN 5UP 5DN"
- board text removed: "5DN 5UP 4DN 4UP"
- board text removed: "IR- IR+"
- board text removed: "L N 1UP 1DN"
- board text removed: "MAR 2025"
- board text removed: "Rev 1.1"
