File: hw-covers.kicad_pcb (KiCad board)
At the start: 2 copper layers, 167 x 100 mm, 147 parts, among them J1 Screw_Terminal_01x04, J10 Screw_Terminal_01x03, J11 Screw_Terminal_01x03, J2 Screw_Terminal_01x04, J3 Conn_01x04_Pin, J4 Conn_01x04_Pin, J5 Screw_Terminal_01x03, J6 Conn_01x02_Pin, J7 Screw_Terminal_01x04, J8 Screw_Terminal_01x03, J9 Screw_Terminal_01x03, K11 SANYOU_SRD_Form_C, K12 SANYOU_SRD_Form_C, K13 SANYOU_SRD_Form_C, K14 SANYOU_SRD_Form_C, K15 SANYOU_SRD_Form_C, K16 SANYOU_SRD_Form_C, K17 SANYOU_SRD_Form_C, K18 SANYOU_SRD_Form_C, K19 SANYOU_SRD_Form_C, K20 SANYOU_SRD_Form_C, Q11 PMBT3904235, Q12 PMBT3904235, Q13 PMBT3904235, Q14 PMBT3904235, Q15 PMBT3904235, Q16 PMBT3904235, Q17 PMBT3904235, Q18 PMBT3904235, Q19 PMBT3904235, Q20 PMBT3904235, Q21 PMBT3904235, SW1 SW_Push, U1 ESP32-S3-WROOM-1, U2 NCP1117-3.3_SOT223

Commit message: Release 2.1.0
Parts:
- added R1: 1k, Resistor_SMD:R_0603_1608Metric, F.Cu at (208.2, 130.0)
- C15, C16, C17, C18, C19, C20, C21, C22, C23, C24: value C -> 100n
- R16, R38, R41, R42, R45, R46, R47, R48, R53, R54: value 1k -> 470
- R39, R40, R43, R44, R49, R50, R51, R52, R55, R56: value R -> 220
- moved Q11 1.50 mm to (208.8, 133.0)
- moved J6 0.50 mm to (214.0, 129.1)
- moved R17 0.29 mm to (208.2, 128.0)
Connections:
- Q11 pad 1: /IR -> Net-(Q11-Pad1)
Routing:
- net /LF: track 288.1 -> 282.3 mm
- net Net-(Q11-Pad1): track 0.00 -> 2.54 mm
- net Net-(J6-Pin_2): track 3.87 -> 5.07 mm
- net Net-(J6-Pin_1): track 4.70 -> 5.46 mm
- net /IR: track 19.3 -> 18.6 mm
- net GND: vias 223 -> 297
Other:
- board text added: "L N 1DN 1UP"
- board text added: "Rev 2.1"
- board text removed: "N L 1DN 1UP"
- board text removed: "Rev 2.0"
