File: inputs.kicad_sch (KiCad schematic)
At the start: 40 parts

Commit message: Add placement
Parts:
- R19, R20, R22, R24, R26, R28, R30, R32, R34, R36: value 10k -> 1k5
Changed lines of the file:
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@@
 			)
 		)
-		(property "Value" "10k"
+		(property "Value" "1k5"
 			(at 140.97 68.58 0)
 			(effects
@@
 			)
 		)
-		(property "Value" "10k"
+		(property "Value" "1k5"
 			(at 73.66 68.58 0)
 			(effects
@@
 			)
 		)
-		(property "Value" "10k"
+		(property "Value" "1k5"
 			(at 73.66 118.11 0)
 			(effects
@@
 			)
 		)
-		(property "Value" "10k"
+		(property "Value" "1k5"
 			(at 205.74 68.58 0)
 			(effects
@@
 			)
 		)
-		(property "Value" "10k"
+		(property "Value" "1k5"
 			(at 166.37 118.11 0)
 			(effects
@@
 			)
 		)
-		(property "Value" "10k"
+		(property "Value" "1k5"
 			(at 231.14 68.58 0)
 			(effects
@@
 			)
 		)
-		(property "Value" "10k"
+		(property "Value" "1k5"
 			(at 99.06 118.11 0)
 			(effects
@@
 			)
 		)
-		(property "Value" "10k"
+		(property "Value" "1k5"
 			(at 140.97 118.11 0)
 			(effects
@@
 			)
 		)
-		(property "Value" "10k"
+		(property "Value" "1k5"
 			(at 166.37 68.58 0)
 			(effects
@@
 			)
 		)
-		(property "Value" "10k"
+		(property "Value" "1k5"
 			(at 99.06 68.58 0)
 			(effects
