File: hw-covers.kicad_sch (KiCad schematic)
At the start: 37 parts, among them J1 Screw_Terminal_01x04, J10 Screw_Terminal_01x03, J11 Screw_Terminal_01x03, J2 Screw_Terminal_01x04, J3 Conn_01x04_Pin, J4 Conn_01x04_Pin, J5 Screw_Terminal_01x03, J6 Conn_01x02_Pin, J7 Screw_Terminal_01x04, J8 Screw_Terminal_01x03, J9 Screw_Terminal_01x03, Q11 PMBT3904235, SW1 SW_Push, U1 ESP32-S3-WROOM-1, U2 NCP1117-3.3_SOT223

Commit message: Finish routing
Connections:
- net 1IN1: now also U1.17 (IO9); no longer U1.22 (IO14)
- net 1IN2: now also U1.18 (IO10); no longer U1.23 (IO21)
- net 2IN1: now also U1.13 (USB_D-); no longer U1.24 (IO47)
- net 2IN2: now also U1.14 (USB_D+); no longer U1.25 (IO48)
- net 3IN1: now also U1.33 (IO40); no longer U1.32 (IO39)
- net 3IN2: now also U1.32 (IO39); no longer U1.33 (IO40)
- net 4IN1: now also U1.35 (IO42); no longer U1.34 (IO41)
- net 4IN2: now also U1.34 (IO41); no longer U1.35 (IO42)
- net 5IN1: now also U1.39 (IO1); no longer U1.38 (IO2)
- net 5IN2: now also U1.38 (IO2); no longer U1.39 (IO1)
- net DIR1: now also U1.19 (IO11); no longer U1.18 (IO10)
- net DIR2: now also U1.21 (IO13); no longer U1.14 (USB_D+)
- net DIR3: now also U1.23 (IO21); no longer U1.12 (IO8)
- net DIR4: now also U1.12 (IO8); no longer U1.10 (IO17)
- net DIR5: now also U1.10 (IO17); no longer U1.8 (IO15)
- net EXT1: now also U1.4 (IO4); no longer U1.5 (IO5)
- net EXT2: now also U1.5 (IO5); no longer U1.4 (IO4)
- net LED1: now also U1.8 (IO15); no longer U1.19 (IO11)
- net LED2: now also U1.7 (IO7); no longer U1.20 (IO12)
- net OUT1: now also U1.20 (IO12); no longer U1.17 (IO9)
- net OUT2: now also U1.22 (IO14); no longer U1.13 (USB_D-)
- net OUT3: now also U1.24 (IO47); no longer U1.11 (IO18)
- net OUT4: now also U1.11 (IO18); no longer U1.9 (IO16)
- net OUT5: now also U1.9 (IO16); no longer U1.7 (IO7)
- net at TP1.1: now also U1.25 (IO48); no longer U1.21 (IO13)
Other:
- moved on the sheet: TP1, TP2
Changed lines of the file:
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@@
 	(wire
 		(pts
+			(xy 205.74 115.57) (xy 213.36 115.57)
+		)
+		(stroke
+			(width 0)
+			(type default)
+		)
+	)
+	(wire
+		(pts
 			(xy 85.09 168.91) (xy 74.93 168.91)
 		)
@@
 	(wire
 		(pts
+			(xy 251.46 102.87) (xy 243.84 102.87)
+		)
+		(stroke
+			(width 0)
+			(type default)
+		)
+	)
+	(wire
+		(pts
 			(xy 143.51 161.29) (xy 133.35 161.29)
 		)
@@
 	)
 	(label "1IN1"
-		(at 205.74 118.11 0)
+		(at 205.74 105.41 0)
 		(effects
 			(font
@@
 	)
 	(label "EXT1"
-		(at 205.74 95.25 0)
+		(at 205.74 92.71 0)
 		(effects
 			(font
@@
 	)
 	(label "DIR3"
-		(at 205.74 102.87 0)
+		(at 251.46 92.71 180)
 		(effects
 			(font
 				(size 1.27 1.27)
 			)
-			(justify left bottom)
+			(justify right bottom)
 		)
 	)
@@
 	)
 	(label "OUT2"
-		(at 251.46 87.63 180)
+		(at 205.74 118.11 0)
 		(effects
 			(font
 				(size 1.27 1.27)
 			)
-			(justify right bottom)
+			(justify left bottom)
 		)
 	)
 	(label "5IN2"
-		(at 205.74 85.09 0)
+		(at 205.74 87.63 0)
 		(effects
 			(font
@@
 	)
 	(label "OUT3"
-		(at 251.46 85.09 180)
+		(at 251.46 120.65 180)
 		(effects
 			(font
@@
 	)
 	(label "DIR1"
-		(at 205.74 107.95 0)
+		(at 205.74 110.49 0)
 		(effects
 			(font
@@
 	)
 	(label "DIR2"
-		(at 251.46 90.17 180)
+		(at 205.74 115.57 0)
 		(effects
 			(font
 				(size 1.27 1.27)
 			)
-			(justify right bottom)
+			(justify left bottom)
 		)
 	)
@@
 	)
 	(label "3IN1"
-		(at 251.46 105.41 180)
+		(at 251.46 107.95 180)
 		(effects
 			(font
@@
 	)
 	(label "OUT1"
-		(at 205.74 105.41 0)
+		(at 205.74 113.03 0)
 		(effects
 			(font
@@
 	)
 	(label "3IN2"
-		(at 251.46 107.95 180)
+		(at 251.46 105.41 180)
 		(effects
 			(font
@@
 	)
 	(label "LED1"
-		(at 205.74 110.49 0)
+		(at 205.74 120.65 0)
 		(effects
 			(font
@@
 	)
 	(label "5IN1"
-		(at 205.74 87.63 0)
+		(at 205.74 85.09 0)
 		(effects
 			(font
@@
 	)
 	(label "LED2"
-		(at 205.74 113.03 0)
+		(at 205.74 100.33 0)
 		(effects
 			(font
@@
 	)
 	(label "4IN2"
-		(at 251.46 113.03 180)
+		(at 251.46 110.49 180)
 		(effects
 			(font
@@
 	)
 	(label "DIR5"
-		(at 205.74 120.65 0)
+		(at 251.46 82.55 180)
 		(effects
 			(font
 				(size 1.27 1.27)
 			)
-			(justify left bottom)
+			(justify right bottom)
 		)
 	)
@@
 	)
 	(label "EXT2"
-		(at 205.74 92.71 0)
+		(at 205.74 95.25 0)
 		(effects
 			(font
@@
 	)
 	(label "OUT5"
-		(at 205.74 100.33 0)
+		(at 205.74 123.19 0)
 		(effects
 			(font
@@
 	)
 	(label "OUT4"
-		(at 205.74 123.19 0)
+		(at 251.46 85.09 180)
 		(effects
 			(font
 				(size 1.27 1.27)
 			)
-			(justify left bottom)
+			(justify right bottom)
 		)
 	)
@@
 	)
 	(label "DIR4"
-		(at 251.46 82.55 180)
+		(at 205.74 102.87 0)
 		(effects
 			(font
 				(size 1.27 1.27)
 			)
-			(justify right bottom)
+			(justify left bottom)
 		)
 	)
 	(label "1IN2"
-		(at 251.46 92.71 180)
+		(at 205.74 107.95 0)
 		(effects
 			(font
 				(size 1.27 1.27)
 			)
-			(justify right bottom)
+			(justify left bottom)
 		)
 	)
@@
 	)
 	(label "2IN2"
-		(at 251.46 123.19 180)
+		(at 251.46 90.17 180)
 		(effects
 			(font
@@
 	)
 	(label "2IN1"
-		(at 251.46 120.65 180)
+		(at 251.46 87.63 180)
 		(effects
 			(font
@@
 	)
 	(label "4IN1"
-		(at 251.46 110.49 180)
+		(at 251.46 113.03 180)
 		(effects
 			(font
@@
 	(symbol
 		(lib_id "Connector:TestPoint")
-		(at 243.84 102.87 270)
+		(at 251.46 102.87 270)
 		(unit 1)
 		(exclude_from_sim no)
@@
 		(dnp no)
 		(property "Reference" "TP2"
-			(at 249.936 102.362 90)
+			(at 257.556 102.362 90)
 			(effects
 				(font
@@
 		)
 		(property "Value" "TestPoint"
-			(at 247.142 105.41 90)
+			(at 254.762 105.41 90)
 			(effects
 				(font
@@
 		)
 		(property "Footprint" "TestPoint:TestPoint_Pad_D1.5mm"
-			(at 243.84 107.95 0)
+			(at 251.46 107.95 0)
 			(effects
 				(font
@@
 		)
 		(property "Datasheet" "~"
-			(at 243.84 107.95 0)
+			(at 251.46 107.95 0)
 			(effects
 				(font
@@
 		)
 		(property "Description" "test point"
-			(at 243.84 102.87 0)
+			(at 251.46 102.87 0)
 			(effects
 				(font
@@
 	(symbol
 		(lib_id "Connector:TestPoint")
-		(at 213.36 115.57 90)
+		(at 251.46 123.19 270)
 		(unit 1)
 		(exclude_from_sim no)
@@
 		(dnp no)
 		(property "Reference" "TP1"
-			(at 207.264 114.808 90)
+			(at 257.556 123.952 90)
 			(effects
 				(font
@@
 		)
 		(property "Value" "TestPoint"
-			(at 210.058 113.03 90)
+			(at 254.762 125.73 90)
 			(effects
 				(font
@@
 		)
 		(property "Footprint" "TestPoint:TestPoint_Pad_D1.5mm"
-			(at 213.36 110.49 0)
+			(at 251.46 128.27 0)
 			(effects
 				(font
@@
 		)
 		(property "Datasheet" "~"
-			(at 213.36 110.49 0)
+			(at 251.46 128.27 0)
 			(effects
 				(font
@@
 		)
 		(property "Description" "test point"
-			(at 213.36 115.57 0)
+			(at 251.46 123.19 0)
 			(effects
 				(font

Commit message: Ready to release
Other:
- note removed: "TODOs: Revisar resistencias entrada"
Changed lines of the file:
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@@
-		)
-	)
-	(text "TODOs:\nRevisar resistencias entrada"
-		(exclude_from_sim no)
-		(at 177.8 168.91 0)
-		(effects
-			(font
-				(size 1.27 1.27)
-			)
-			(justify left)
 		)
 	)

Commit message: Release 2.1.0
Parts:
- added R1: 1k, Resistor_SMD:R_0603_1608Metric, symbol Device:R
Connections:
- net IR: now also R1.1; no longer Q11.1
- new net: Q11.1, R1.2
Changed lines of the file:
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@@
 	(title_block
 		(title "Covers")
-		(date "2026-03-08")
-		(rev "Rev 2.0")
+		(date "2026-03-09")
+		(rev "Rev 2.1")
 		(company "Guille González")
 	)
@@
 	(wire
 		(pts
-			(xy 123.19 110.49) (xy 128.27 110.49)
+			(xy 111.76 110.49) (xy 118.11 110.49)
 		)
 		(stroke
@@
 		(pts
 			(xy 39.37 36.83) (xy 40.64 36.83)
+		)
+		(stroke
+			(width 0)
+			(type default)
+		)
+	)
+	(wire
+		(pts
+			(xy 125.73 110.49) (xy 128.27 110.49)
 		)
 		(stroke
@@
 	)
 	(label "IR"
-		(at 123.19 110.49 0)
+		(at 111.76 110.49 0)
 		(effects
 			(font
@@
 					(unit 1)
 				)
+			)
+		)
+	)
+	(symbol
+		(lib_id "Device:R")
+		(at 121.92 110.49 90)
+		(unit 1)
+		(exclude_from_sim no)
+		(in_bom yes)
+		(on_board yes)
+		(dnp no)
+		(property "Reference" "R1"
+			(at 120.65 107.95 90)
+			(effects
+				(font
+					(size 1.27 1.27)
+				)
+			)
+		)
+		(property "Value" "1k"
+			(at 124.46 107.95 90)
+			(effects
+				(font
+					(size 1.27 1.27)
+				)
+			)
+		)
+		(property "Footprint" "Resistor_SMD:R_0603_1608Metric"
+			(at 121.92 112.268 90)
+			(effects
+				(font
+					(size 1.27 1.27)
+				)
+				(hide yes)
+			)
+		)
+		(property "Datasheet" "~"
+			(at 121.92 110.49 0)
+			(effects
+				(font
+					(size 1.27 1.27)
+				)
+				(hide yes)
+			)
+		)
+		(property "Description" "Resistor"
+			(at 121.92 110.49 0)
+			(effects
+				(font
+					(size 1.27 1.27)
+				)
+				(hide yes)
+			)
+		)
+		(pin "1"
+		)
+		(pin "2"
+		)
+		(instances
+			(project "hw-covers"
+				(path "/7d538877-0678-43a6-9ffb-51bd93bb2c44"
+					(reference "R1")
+					(unit 1)
+				)
