File: outputs.kicad_sch (KiCad schematic)
At the start: 70 parts, among them K11 SANYOU_SRD_Form_C, K12 SANYOU_SRD_Form_C, K13 SANYOU_SRD_Form_C, K14 SANYOU_SRD_Form_C, K15 SANYOU_SRD_Form_C, K16 SANYOU_SRD_Form_C, K17 SANYOU_SRD_Form_C, K18 SANYOU_SRD_Form_C, K19 SANYOU_SRD_Form_C, K20 SANYOU_SRD_Form_C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

Commit message: Add placement
Other:
- moved on the sheet: D29, K16, Q17, R46

Commit message: Release 2.1.0
Parts:
- C15, C16, C17, C18, C19, C20, C21, C22, C23, C24: value C -> 100n
- R16, R38, R41, R42, R45, R46, R47, R48, R53, R54: value 1k -> 470
- R39, R40, R43, R44, R49, R50, R51, R52, R55, R56: value R -> 220
Changed lines of the file:
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@@
 			)
 		)
-		(property "Value" "1k"
+		(property "Value" "470"
 			(at 109.982 87.63 0)
 			(effects
@@
 		(dnp no)
 		(property "Reference" "C17"
-			(at 133.35 26.924 90)
+			(at 130.81 26.67 90)
 			(effects
 				(font
@@
 			)
 		)
-		(property "Value" "C"
+		(property "Value" "100n"
 			(at 135.89 26.924 90)
 			(effects
@@
 			)
 		)
-		(property "Value" "R"
-			(at 222.504 43.434 90)
+		(property "Value" "220"
+			(at 224.79 44.45 90)
 			(effects
 				(font
@@
 			)
 		)
-		(property "Value" "R"
-			(at 143.764 43.434 90)
+		(property "Value" "220"
+			(at 146.05 44.45 90)
 			(effects
 				(font
@@
 			)
 		)
-		(property "Value" "R"
-			(at 183.134 43.434 90)
+		(property "Value" "220"
+			(at 185.42 44.45 90)
 			(effects
 				(font
@@
 			)
 		)
-		(property "Value" "R"
-			(at 183.134 26.924 90)
+		(property "Value" "220"
+			(at 185.42 27.94 90)
 			(effects
 				(font
@@
 		(dnp no)
 		(property "Reference" "C23"
-			(at 57.15 26.924 90)
+			(at 54.61 26.67 90)
 			(effects
 				(font
@@
 			)
 		)
-		(property "Value" "C"
+		(property "Value" "100n"
 			(at 59.69 26.924 90)
 			(effects
@@
 			)
 		)
-		(property "Value" "R"
-			(at 222.504 26.924 90)
+		(property "Value" "220"
+			(at 224.79 27.94 90)
 			(effects
 				(font
@@
 		(dnp no)
 		(property "Reference" "C22"
-			(at 212.09 43.434 90)
+			(at 209.55 43.18 90)
 			(effects
 				(font
@@
 			)
 		)
-		(property "Value" "C"
+		(property "Value" "100n"
 			(at 214.63 43.434 90)
 			(effects
@@
 		(dnp no)
 		(property "Reference" "C15"
-			(at 95.25 43.434 90)
+			(at 92.71 43.18 90)
 			(effects
 				(font
@@
 			)
 		)
-		(property "Value" "C"
+		(property "Value" "100n"
 			(at 97.79 43.434 90)
 			(effects
@@
 			)
 		)
-		(property "Value" "R"
-			(at 67.564 26.924 90)
+		(property "Value" "220"
+			(at 69.85 27.94 90)
 			(effects
 				(font
@@
 			)
 		)
-		(property "Value" "1k"
+		(property "Value" "470"
 			(at 178.562 115.57 0)
 			(effects
@@
 		(dnp no)
 		(property "Reference" "C18"
-			(at 133.35 43.434 90)
+			(at 130.81 43.18 90)
 			(effects
 				(font
@@
 			)
 		)
-		(property "Value" "C"
+		(property "Value" "100n"
 			(at 135.89 43.434 90)
 			(effects
@@
 			)
 		)
-		(property "Value" "1k"
+		(property "Value" "470"
 			(at 41.402 115.57 0)
 			(effects
@@
 		(dnp no)
 		(property "Reference" "C16"
-			(at 95.25 26.924 90)
+			(at 92.71 26.67 90)
 			(effects
 				(font
@@
 			)
 		)
-		(property "Value" "C"
+		(property "Value" "100n"
 			(at 97.79 26.924 90)
 			(effects
@@
 			)
 		)
-		(property "Value" "1k"
+		(property "Value" "470"
 			(at 41.402 176.53 0)
 			(effects
@@
 			)
 		)
-		(property "Value" "1k"
+		(property "Value" "470"
 			(at 178.562 87.63 0)
 			(effects
@@
 		(dnp no)
 		(property "Reference" "C21"
-			(at 212.09 26.924 90)
+			(at 209.55 26.67 90)
 			(effects
 				(font
@@
 			)
 		)
-		(property "Value" "C"
+		(property "Value" "100n"
 			(at 214.63 26.924 90)
 			(effects
@@
 			)
 		)
-		(property "Value" "1k"
+		(property "Value" "470"
 			(at 109.982 115.57 0)
 			(effects
@@
 			)
 		)
-		(property "Value" "R"
-			(at 105.664 26.924 90)
+		(property "Value" "220"
+			(at 107.95 27.94 90)
 			(effects
 				(font
@@
 		(dnp no)
 		(property "Reference" "C24"
-			(at 57.15 43.434 90)
+			(at 54.61 43.18 90)
 			(effects
 				(font
@@
 			)
 		)
-		(property "Value" "C"
+		(property "Value" "100n"
 			(at 59.69 43.434 90)
 			(effects
@@
 		(dnp no)
 		(property "Reference" "C19"
-			(at 172.72 26.924 90)
+			(at 170.18 26.67 90)
 			(effects
 				(font
@@
 			)
 		)
-		(property "Value" "C"
+		(property "Value" "100n"
 			(at 175.26 26.924 90)
 			(effects
@@
 			)
 		)
-		(property "Value" "R"
-			(at 105.664 43.434 90)
+		(property "Value" "220"
+			(at 107.95 44.45 90)
 			(effects
 				(font
@@
 			)
 		)
-		(property "Value" "1k"
+		(property "Value" "470"
 			(at 109.982 176.53 0)
 			(effects
@@
 			)
 		)
-		(property "Value" "1k"
+		(property "Value" "470"
 			(at 41.402 148.59 0)
 			(effects
@@
 			)
 		)
-		(property "Value" "R"
-			(at 143.764 26.924 90)
+		(property "Value" "220"
+			(at 146.05 27.94 90)
 			(effects
 				(font
@@
 			)
 		)
-		(property "Value" "1k"
+		(property "Value" "470"
 			(at 41.402 87.63 0)
 			(effects
@@
 			)
 		)
-		(property "Value" "R"
-			(at 67.564 43.434 90)
+		(property "Value" "220"
+			(at 69.85 44.45 90)
 			(effects
 				(font
@@
 			)
 		)
-		(property "Value" "1k"
+		(property "Value" "470"
 			(at 109.982 149.86 0)
 			(effects
@@
 		(dnp no)
 		(property "Reference" "C20"
-			(at 172.72 43.434 90)
+			(at 170.18 43.18 90)
 			(effects
 				(font
@@
 			)
 		)
-		(property "Value" "C"
+		(property "Value" "100n"
 			(at 175.26 43.434 90)
 			(effects
